File: Beta1/Keys/_autosave-Keyboard_Pads.kicad_pcb (KiCad board)
At the start: 2 copper layers, 194 x 64.2 mm, 28 parts, among them U1 MPR121TH

Commit message: Add MPR
Parts:
- moved U1 95.1 mm to (6.69, -19.9)
Changed lines of the file:
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@@
   )
   (module Liberry:MPR121TH (layer F.Cu)
-    (at 96.98 10.050001)
+    (at 6.69 -19.905)
     (fp_text reference U1 (at 1.27 -2.54) (layer F.SilkS)
       (effects (font (size 1 1) (thickness 0.15)))
