File: Beta1/Wanderlust.sch (KiCad schematic (older format))
At the start: 26 parts, among them P0 CONN_01X01, P1 CONN_01X01, P10 CONN_01X01, P11 CONN_01X01, P2 CONN_01X01, P3 CONN_01X01, P4 CONN_01X01, P5 CONN_01X01, P6 CONN_01X01, P7 CONN_01X01, P8 CONN_01X01, P9 CONN_01X01, U1 MPR121QR2

Commit message: Catchup Commit.  Non-atomic, Refactored LED, Keyboard, KeyPAD, and Knobs PCBs
LED: Changed chips. Cleaned up silkscreen text. Added some support
mounting holes. Shrank height of board to avoid stackup. KeyPAD is
updated with new footprint. Keyboard and Knobs are unknown.
Parts:
- U1: footprint Liberry:QFN-20-1EP_3x3mm_Pitch0.65mm -> Liberry:QFN-20-1EP_3x3mm_Pitch0.40mm
Changed lines of the file:
@@
 F 0 "U1" H 8150 3650 60  0000 C CNN
 F 1 "MPR121QR2" H 8650 200 60  0000 C CNN
-F 2 "Liberry:QFN-20-1EP_3x3mm_Pitch0.65mm" H 6100 3450 60  0001 C CNN
+F 2 "Liberry:QFN-20-1EP_3x3mm_Pitch0.40mm" H 6100 3450 60  0001 C CNN
 F 3 "" H 6100 3450 60  0001 C CNN
 	1    8050 2650
