File: Beta1/JoyXYMezanine/JoyXYMezanine.sch (KiCad schematic (older format))
At the start: 14 parts

Commit message: Cloned 2CH Joy Mez and replaced a Joy with a knob (volume)
Changed lines of the file:
@@
 $EndComp
 $Comp
-L GND #PWR2
+L GND #PWR01
 U 1 1 582E3FD0
 P 9000 1450
-F 0 "#PWR2" H 9000 1200 50  0001 C CNN
+F 0 "#PWR01" H 9000 1200 50  0001 C CNN
 F 1 "GND" H 9000 1300 50  0000 C CNN
 F 2 "" H 9000 1450 50  0000 C CNN
@@
 $EndComp
 $Comp
-L VCC #PWR1
+L VCC #PWR02
 U 1 1 586B0608
 P 9000 850
-F 0 "#PWR1" H 9000 700 50  0001 C CNN
+F 0 "#PWR02" H 9000 700 50  0001 C CNN
 F 1 "VCC" H 9000 1000 50  0000 C CNN
 F 2 "" H 9000 850 50  0000 C CNN
@@
 	9000 900  8950 900
 $Comp
-L GND #PWR4
+L GND #PWR03
 U 1 1 586B0C2D
 P 12950 3500
-F 0 "#PWR4" H 12950 3250 50  0001 C CNN
+F 0 "#PWR03" H 12950 3250 50  0001 C CNN
 F 1 "GND" H 12950 3350 50  0000 C CNN
 F 2 "" H 12950 3500 50  0000 C CNN
@@
 $EndComp
 $Comp
-L GND #PWR5
+L GND #PWR04
 U 1 1 586B0C53
 P 13100 6150
-F 0 "#PWR5" H 13100 5900 50  0001 C CNN
+F 0 "#PWR04" H 13100 5900 50  0001 C CNN
 F 1 "GND" H 13100 6000 50  0000 C CNN
 F 2 "" H 13100 6150 50  0000 C CNN
@@
 $EndComp
 Wire Wire Line
-	13300 6100 13200 6100
-Wire Wire Line
-	13200 6100 13100 6100
+	13100 6100 13300 6100
 Wire Wire Line
 	13100 6100 13100 6150
 Wire Wire Line
-	12950 3450 13150 3450
-Wire Wire Line
-	13150 3450 13250 3450
+	12950 3450 13250 3450
 Wire Wire Line
 	12950 3450 12950 3500
@@
 $EndComp
 $Comp
-L VCC #PWR3
+L VCC #PWR05
 U 1 1 586B1045
 P 12550 2350
-F 0 "#PWR3" H 12550 2200 50  0001 C CNN
+F 0 "#PWR05" H 12550 2200 50  0001 C CNN
 F 1 "VCC" H 12550 2500 50  0000 C CNN
 F 2 "" H 12550 2350 50  0000 C CNN
@@
 $EndComp
 Wire Wire Line
-	12550 2350 12550 2400
-Wire Wire Line
-	12550 2400 12550 2950
-Wire Wire Line
-	12550 2950 12550 5050
-Wire Wire Line
-	12550 5050 12550 5600
+	12550 2350 12550 5600
 Wire Wire Line
 	12550 2400 13250 2400
@@
 	13250 2700 13150 2700
 Wire Wire Line
-	13150 2700 13150 3250
-Wire Wire Line
-	13150 3250 13150 3450
+	13150 2700 13150 3450
 Connection ~ 13150 3450
 Wire Wire Line
@@
 	13300 5350 13200 5350
 Wire Wire Line
-	13200 5350 13200 5900
-Wire Wire Line
-	13200 5900 13200 6100
+	13200 5350 13200 6100
 Connection ~ 13200 6100
 Wire Wire Line
