File: Beta1/PCB1001_LED32/PCB1002_LED32.sch (KiCad schematic (older format))
At the start: 220 parts, among them U0 APA102C, U1 APA102C, U10 APA102C, U11 APA102C, U12 APA102C, U13 APA102C, U14 APA102C, U15 APA102C, U16 APA102C, U17 APA102C, U18 APA102C, U19 APA102C, U2 APA102C, U20 APA102C, U21 APA102C, U22 APA102C, U23 APA102C, U24 APA102C, U25 APA102C, U26 APA102C, U27 APA102C, U28 APA102C, U29 APA102C, U3 APA102C, U30 APA102C, U31 APA102C, U4 APA102C, U5 APA102C, U6 APA102C, U7 APA102C, U8 APA102C, U9 APA102C

Commit message: Removed jumper resistors, b/c as they cause shorts.
Parts:
- removed D0: CONN_01X01, Liberry:single_0.1, symbol CONN_01X01
- removed D1, D2, D3, D4, D5, D6, D7: CONN_01X01, Liberry:TESTPAD, symbol CONN_01X01
- removed RC0, RC1, RC10, RC11, RC12, RC13, RC14, RC15, RC16, RC17, RC18, RC19, RC2, RC20, RC21, RC22, RC23, RC24, RC25, RC26, RC27, RC28, RC29, RC3, RC30, RC31, RC4, RC5, RC6, RC7, RC8, RC9, RD0, RD1, RD10, RD11, RD12, RD13, RD14, RD15, RD16, RD17, RD18, RD19, RD2, RD20, RD21, RD22, RD23, RD24, RD25, RD26, RD27, RD28, RD29, RD3, RD30, RD31, RD4, RD5, RD6, RD7, RD8, RD9: ZERO, Resistors_SMD:R_0603, symbol R
Connections:
- wire segments 579 -> 315
