File: Beta1/PCB1002_1Octave_16PAD/PCB1002_1Octave_16PAD.kicad_pcb (KiCad board)
At the start: 2 copper layers, 188.9 x 64 mm, 98 parts, among them P0 CONN_01X01, P1 CONN_01X01, P10 CONN_01X01, P100 CONN_01X01, P101 CONN_01X01, P102 CONN_01X01, P103 CONN_01X01, P104 CONN_01X01, P105 CONN_01X01, P106 CONN_01X01, P107 CONN_01X01, P108 CONN_01X01, P109 CONN_01X01, P11 CONN_01X01, P110 CONN_01X01, P111 CONN_01X01, P2 CONN_01X01, P200 CONN_01X01, P201 CONN_01X01, P202 CONN_01X01, P203 CONN_01X01, P204 CONN_01X01, P205 CONN_01X01, P206 CONN_01X01, P207 CONN_01X01, P208 CONN_01X01, P209 CONN_01X01, P210 CONN_01X01, P211 CONN_01X01, P3 CONN_01X01, P4 CONN_01X01, P5 CONN_01X01, P6 CONN_01X01, P7 CONN_01X01, P8 CONN_01X01, P9 CONN_01X01, U1 MPR121QR2, U100 MPR121QR2, U200 MPR121QR2

Commit message: Renamed to 1Octave
Other:
- board text added: "PCB1002_1OCTAVE_16PAD_2017-01-26 Beta-1 Believotron Wanderlust 1/2 H Keypad 1 Octave Piano, 16 Pads 6CH Analog Mezzanine Expansion headers"
- board text removed: "PCB1002_Piano_16PAD_2017-01-26 Beta-1 Believotron Wanderlust 1/2 H Keypad 1 Octave Piano, 16 Pads 6CH Analog Mezzanine Expansion headers"
Changed lines of the file:
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@@
     (links 128)
     (no_connects 0)
-    (area 2.489999 -64.160001 191.470001 -0.089999)
+    (area -10.627639 -69.5074 191.470001 7.9024)
     (thickness 1.6)
     (drawings 57)
@@
       (net 32 "Net-(P111-Pad1)"))
   )
-  (gr_text "Open Source License at:\nhttps://github.com/Believotron/BelievotronWanderlustHardware\n\nMarketing pap: \nbelievotron.com\n\nThe good stuff:\nhttp://community.believotron.com/" (at 18.288 -21.844 90) (layer F.SilkS)
+  (gr_text "Open Source License at:\nhttps://github.com/Believotron/BelievotronWanderlustHardware\n\nMarketing pap: \nbelievotron.com\n\nThe good stuff:\nhttp://community.believotron.com/" (at 18.542 -21.844 90) (layer F.SilkS)
     (effects (font (size 0.45 0.45) (thickness 0.1125)) (justify left))
   )
@@
     (effects (font (size 0.75 0.75) (thickness 0.1875)) (justify mirror))
   )
-  (gr_text "PCB1002_Piano_16PAD_2017-01-26 Beta-1\nBelievotron Wanderlust 1/2 H Keypad\n1 Octave Piano, 16 Pads\n6CH Analog Mezzanine Expansion headers" (at 7.62 -37.592 90) (layer F.SilkS)
+  (gr_text "PCB1002_1OCTAVE_16PAD_2017-01-26 Beta-1\nBelievotron Wanderlust 1/2 H Keypad\n1 Octave Piano, 16 Pads\n6CH Analog Mezzanine Expansion headers" (at 7.62 -37.592 90) (layer F.SilkS)
     (effects (font (size 0.6 0.6) (thickness 0.15)) (justify left))
   )
