File: Beta1/PCB1004_Wanderlust_Axoloti_Translator/PCB1004_Wanderlust_Axoloti_Translator.sch (KiCad schematic (older format))
At the start: 93 parts, among them U1 CPT112S, U100 CPT112S, U200 CPT112S

Commit message: First pass schematic on translator board.
Parts:
- removed C1, C101, C201: 0.1uf, Capacitors_SMD:C_0603, symbol C
- removed C102, C2, C202: 4.7 uF, Capacitors_SMD:C_0603, symbol C
- removed CFG_CLK_U1, CFG_CLK_U100, CFG_CLK_U200, CFG_DAT_U1, CFG_DAT_U100, CFG_DAT_U200, GND_U1, GND_U100, GND_U200, PD0, PD1, PD100, PD101, PD102, PD103, PD2, PD3: CONN_01X01, Liberry:single_0.1, symbol CONN_01X01
- removed PAD0, PAD1, PAD100, PAD101, PAD102, PAD103, PAD104, PAD105, PAD106, PAD107, PAD3, PAD4, PAD5, PAD6, PAD7: TOUCHPAD_10CM, Liberry:TOUCH_PAD_10CM, symbol TOUCHPAD_10CM
- removed PAD2: TOUCHPAD_10CM, Liberry:TOUCH_PAD_10CM_V2, symbol TOUCHPAD_10CM
- removed TP0, TP1, TP10, TP100, TP101, TP102, TP103, TP104, TP105, TP106, TP107, TP108, TP109, TP11, TP110, TP111, TP2, TP200, TP201, TP202, TP203, TP204, TP205, TP206, TP207, TP208, TP209, TP210, TP211, TP3, TP4, TP5, TP6, TP7, TP8, TP9: CONN_01X01, Liberry:TESTPAD, symbol CONN_01X01
- removed U1, U100, U200: CPT112S, Liberry:SOIC-24_0.635_1.5x5.2, symbol CPT112S
- removed UKEY0: KEYBOARD_1OCT, Liberry:Keyboard_1_Octave_20CM, symbol KEYBOARD_1OCT
- added +3.3V_LED0, GND_LED0, KNOB_+3.3V0, KNOB_GND0, KNOB_JOY_SW0, KNOB_JOY_X0, KNOB_JOY_Y0, KNOB_SPI_CLK0, KNOB_SPI_CS_0_7, KNOB_SPI_CS_8_15, KNOB_SPI_MISO0, KNOB_SPI_MOSI0, KNOB_VOL0, SPI_CLK_LED0, SPI_MOSI_LED_0: CONN_01X01, Liberry:TH_0.1_1x2_Jumper, symbol CONN_01X01
- added J?: Axoloti_40Pin, Liberry:Axoloti-40x3, symbol Axoloti_40Pin
Connections:
- net labels added: ANALOG_OUT, I2C_SCL, I2C_SDA, JOY_SW, JOY_X, JOY_Y, KB_A0, KB_A1, KB_A2, KB_A3, KB_A4, KB_A5, KB_IRQ, KNOB_CS_0_7, KNOB_CS_8_15, SPI_CLK, SPI_CS_LED0, SPI_MISO, SPI_MOSI, VCCA, VCC_A, VCC_B, VCC_C, VOLUME
- net labels removed: +3.3V, CHIP_04, CHIP_05, CHIP_06, CHIP_07, CHIP_08, CHIP_09, CHIP_10, CHIP_104, CHIP_105, CHIP_106, CHIP_107, CHIP_108, CHIP_109, CHIP_11, CHIP_110, CHIP_111, CHIP_200, CHIP_201, CHIP_202, CHIP_203, CHIP_204, CHIP_205, CHIP_206, CHIP_207, CHIP_208, CHIP_209, CHIP_210, CHIP_211, IRQ, SCL, SDA
- wire segments 194 -> 71
Other:
- note added: "PCB1000_16CH_KNOB+JOY+VOL\nConnector"
- note added: "PCB1001_LED32\nConnector"
- note added: "PCB1003_CPT112S\nConnector"
- note removed: "The Pad to Chip connections are backdriven by the physics of the capacitance touch-chip. \nIn order to minimize interference between traces, we must alternate them. \nThe low cost of the sensor and it's suitability in a field of competitors, \ncoupled with the chip configuration tradeoffs to achieve HMI realtime feel \nrequires that we break best practice of making the data labels match the bit o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"
- moved on the sheet: +3.3V0, A0, A1, A2, A3, A4, A5, GND0, IRQ0, R301, R302, R303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

Commit message: Fixed small bugs, cleaned up the graphics
Parts:
- added KNOB_ANALOG_OUT0, SPI_CS_LED0: CONN_01X01, Liberry:TH_0.1_1x2_Jumper, symbol CONN_01X01
- gave numbers to parts that had none: 1
Connections:
- net labels removed: VCCA
- wire segments 71 -> 73
Other:
- note added: "Believotron Wanderlust Beta 1 to Axoloti Core v1.1 translator board"
- note added: "Believotron Wanderlust Beta1 to Axoloti v1.1 translator PCB"
- note removed: "Believotron Wanderlust 16 Keypay, 1 Octave Piano Cap touch pad to I2C"
Changed lines of the file:
@@
 $EndComp
 $Comp
-L GND #PWR02
+L GND #PWR01
 U 1 1 582F5B3F
 P 1600 1050
-F 0 "#PWR02" H 1600 800 50  0001 C CNN
+F 0 "#PWR01" H 1600 800 50  0001 C CNN
 F 1 "GND" H 1600 900 50  0000 C CNN
 F 2 "" H 1600 1050 50  0000 C CNN
@@
 DATE
 Text Notes 29650 21250 0    60   ~ 0
-Believotron Wanderlust 16 Keypay, 1 Octave Piano Cap touch pad to I2C
-$Comp
-L Axoloti_40Pin J?
+Believotron Wanderlust Beta1 to Axoloti v1.1 translator PCB
+$Comp
+L Axoloti_40Pin J1
 U 1 1 58DEE951
 P 11250 7000
-F 0 "J?" H 11550 12500 60  0000 C CNN
+F 0 "J1" H 11550 12500 60  0000 C CNN
 F 1 "Axoloti_40Pin" H 12900 12550 60  0000 C CNN
 F 2 "Liberry:Axoloti-40x3" H 7800 9950 60  0001 C CNN
@@
 PCB1003_CPT112S\nConnector
 Wire Wire Line
-	10600 4650 11250 4650
-Text Label 10650 4650 0    60   ~ 0
+	10400 4650 11250 4650
+Text Label 10450 4650 0    60   ~ 0
 KB_IRQ
 Wire Wire Line
-	11250 2450 10700 2450
-Wire Wire Line
-	11250 2350 10700 2350
-Text Label 10750 2350 0    60   ~ 0
+	10400 2450 11250 2450
+Wire Wire Line
+	10400 2350 11250 2350
+Text Label 10450 2350 0    60   ~ 0
 I2C_SCL
-Text Label 10750 2450 0    60   ~ 0
+Text Label 10450 2450 0    60   ~ 0
 I2C_SDA
-Text Label 10750 2050 0    60   ~ 0
+Text Label 10450 2050 0    60   ~ 0
 VCC_A
 Wire Wire Line
-	10700 2050 11250 2050
+	10400 2050 11250 2050
 Wire Wire Line
 	1850 2250 3250 2250
@@
 Connection ~ 2500 2250
 Text Label 2700 2250 0    60   ~ 0
-VCCA
+VCC_A
 Wire Wire Line
 	2600 800  2600 2250
@@
 KB_A5
 Wire Wire Line
-	10550 2950 11250 2950
-Wire Wire Line
-	10550 3050 11250 3050
-Wire Wire Line
-	10550 3150 11250 3150
-Wire Wire Line
-	10550 3550 11250 3550
-Wire Wire Line
-	10550 3750 11250 3750
-Wire Wire Line
-	10550 3850 11250 3850
-Text Label 10650 2950 0    60   ~ 0
+	10400 2950 11250 2950
+Wire Wire Line
+	10400 3050 11250 3050
+Wire Wire Line
+	10400 3150 11250 3150
+Wire Wire Line
+	10400 3550 11250 3550
+Wire Wire Line
+	10400 3750 11250 3750
+Wire Wire Line
+	10400 3850 11250 3850
+Text Label 10450 2950 0    60   ~ 0
 KB_A0
-Text Label 10650 3050 0    60   ~ 0
+Text Label 10450 3050 0    60   ~ 0
 KB_A1
-Text Label 10650 3150 0    60   ~ 0
+Text Label 10450 3150 0    60   ~ 0
 KB_A2
-Text Label 10650 3550 0    60   ~ 0
+Text Label 10450 3550 0    60   ~ 0
 KB_A3
-Text Label 10650 3750 0    60   ~ 0
+Text Label 10450 3750 0    60   ~ 0
 KB_A4
-Text Label 10650 3850 0    60   ~ 0
+Text Label 10450 3850 0    60   ~ 0
 KB_A5
 $Comp
-L GND #PWR?
+L GND #PWR02
 U 1 1 58DF1717
 P 10250 6250
-F 0 "#PWR?" H 10250 6000 50  0001 C CNN
+F 0 "#PWR02" H 10250 6000 50  0001 C CNN
 F 1 "GND" H 10250 6100 50  0000 C CNN
 F 2 "" H 10250 6250 50  0000 C CNN
@@
 PCB1001_LED32\nConnector
 Wire Wire Line
-	11250 2650 10700 2650
-Text Label 10750 2650 0    60   ~ 0
+	10400 2650 11250 2650
+Text Label 10450 2650 0    60   ~ 0
 VCC_A
 Wire Wire Line
-	11250 3450 10700 3450
-Text Label 10750 3450 0    60   ~ 0
+	10400 3450 11250 3450
+Text Label 10450 3450 0    60   ~ 0
 VCC_B
 Wire Wire Line
-	11250 4050 10700 4050
-Text Label 10750 4050 0    60   ~ 0
+	10400 4050 11250 4050
+Text Label 10450 4050 0    60   ~ 0
 VCC_B
 Wire Wire Line
-	11250 4850 10700 4850
+	10400 4850 11250 4850
 Wire Wire Line
 	11250 4950 11150 4950
@@
 	11150 4950 11150 4850
 Connection ~ 11150 4850
-Text Label 10750 4850 0    60   ~ 0
+Text Label 10450 4850 0    60   ~ 0
 VCC_C
 Wire Wire Line
@@
 	4500 5550 5250 5550
 Wire Wire Line
-	10500 3250 11250 3250
+	10400 3250 11250 3250
 Wire Wire Line
 	4500 5950 5250 5950
 $Comp
-L GND #PWR?
+L GND #PWR03
 U 1 1 58DF4774
 P 4600 6250
-F 0 "#PWR?" H 4600 6000 50  0001 C CNN
+F 0 "#PWR03" H 4600 6000 50  0001 C CNN
 F 1 "GND" H 4600 6100 50  0000 C CNN
 F 2 "" H 4600 6250 50  0000 C CNN
@@
 Text Label 4600 5550 0    60   ~ 0
 SPI_MOSI
-Text Label 10600 3250 0    60   ~ 0
+Text Label 10450 3250 0    60   ~ 0
 SPI_CS_LED0
 Text Label 4600 5950 0    60   ~ 0
 SPI_CLK
 Wire Wire Line
-	11250 4250 10700 4250
-Wire Wire Line
-	11250 4350 10700 4350
-Wire Wire Line
-	11250 4450 10700 4450
-Text Label 10750 4450 0    60   ~ 0
+	10400 4250 11250 4250
+Wire Wire Line
+	10400 4350 11250 4350
+Wire Wire Line
+	10400 4450 11250 4450
+Text Label 10450 4450 0    60   ~ 0
 SPI_MOSI
-Text Label 10750 4350 0    60   ~ 0
+Text Label 10450 4350 0    60   ~ 0
 SPI_MISO
-Text Label 10750 4250 0    60   ~ 0
+Text Label 10450 4250 0    60   ~ 0
 SPI_CLK
 $Comp
@@
 SPI_CLK
 $Comp
-L GND #PWR?
+L GND #PWR04
 U 1 1 58DF831F
 P 6800 5600
-F 0 "#PWR?" H 6800 5350 50  0001 C CNN
+F 0 "#PWR04" H 6800 5350 50  0001 C CNN
 F 1 "GND" H 6800 5450 50  0000 C CNN
 F 2 "" H 6800 5600 50  0000 C CNN
@@
 JOY_SW
 Wire Wire Line
-	10600 2750 11250 2750
-Wire Wire Line
-	10600 2850 11250 2850
-Wire Wire Line
-	10600 4550 11250 4550
-Text Label 10700 2750 0    60   ~ 0
+	10400 2750 11250 2750
+Wire Wire Line
+	10400 2850 11250 2850
+Wire Wire Line
+	10400 4550 11250 4550
+Text Label 10450 2750 0    60   ~ 0
 JOY_Y
-Text Label 10700 2850 0    60   ~ 0
+Text Label 10450 2850 0    60   ~ 0
 JOY_X
-Text Label 10650 4550 0    60   ~ 0
+Text Label 10450 4550 0    60   ~ 0
 JOY_SW
 Wire Wire Line
-	10600 3650 11250 3650
-Wire Wire Line
-	10450 2250 11250 2250
-Wire Wire Line
-	10450 2150 11250 2150
-Text Label 10700 3650 0    60   ~ 0
+	10400 3650 11250 3650
+Wire Wire Line
+	10400 2250 11250 2250
+Wire Wire Line
+	10400 2150 11250 2150
+Text Label 10450 3650 0    60   ~ 0
 VOLUME
-Text Label 10600 2250 0    60   ~ 0
+Text Label 10450 2250 0    60   ~ 0
 KNOB_CS_0_7
-Text Label 10550 2150 0    60   ~ 0
+Text Label 10450 2150 0    60   ~ 0
 KNOB_CS_8_15
 Wire Wire Line
-	10500 4150 11250 4150
-Text Label 10600 4150 0    60   ~ 0
+	10400 4150 11250 4150
+Text Label 10450 4150 0    60   ~ 0
 ANALOG_OUT
+Text Notes 3650 1000 0    157  ~ 0
+Believotron Wanderlust Beta 1 to Axoloti Core v1.1 translator board
+$Comp
+L CONN_01X01 SPI_CS_LED0
+U 1 1 58E01195
+P 4300 5750
+F 0 "SPI_CS_LED0" H 4850 5750 50  0000 R CNN
+F 1 "CONN_01X01" V 4400 5750 50  0001 C CNN
+F 2 "Liberry:TH_0.1_1x2_Jumper" H 4300 5750 50  0001 C CNN
+F 3 "" H 4300 5750 50  0000 C CNN
+F 4 "PCB" H 4300 5750 60  0001 C CNN "MFG"
+F 5 "ON_PCB" H 4300 5750 60  0001 C CNN "MPN"
+	1    4300 5750
+	-1   0    0    1
+$EndComp
+Text Label 4600 5750 0    60   ~ 0
+SPI_CS_LED0
+Wire Wire Line
+	4500 5750 5250 5750
+$Comp
+L CONN_01X01 KNOB_ANALOG_OUT0
+U 1 1 58E02046
+P 6450 3600
+F 0 "KNOB_ANALOG_OUT0" H 7300 3600 50  0000 R CNN
+F 1 "CONN_01X01" V 6550 3600 50  0001 C CNN
+F 2 "Liberry:TH_0.1_1x2_Jumper" H 6450 3600 50  0001 C CNN
+F 3 "" H 6450 3600 50  0000 C CNN
+F 4 "PCB" H 6450 3600 60  0001 C CNN "MFG"
+F 5 "ON_PCB" H 6450 3600 60  0001 C CNN "MPN"
+	1    6450 3600
+	-1   0    0    1
+$EndComp
+Text Label 6750 3600 0    60   ~ 0
+ANALOG_OUT
+Wire Wire Line
+	6650 3600 7400 3600
 $EndSCHEMATC

Commit message: Rough placement complete
Parts:
- renumbered +3.3V0 to KB_+3.3V0, A0 to KB_A0, A1 to KB_A1, A2 to KB_A2, A3 to KB_A3, A4 to KB_A4, A5 to KB_A5, GND0 to KB_GND0, IRQ0 to KB_IRQ0, SCL0 to KB_SCL0, SDA0 to KB_SDA0, +3.3V_LED0 to LED_+3.3V0, GND_LED0 to LED_GND0, SPI_CLK_LED0 to LED_SPI_CLK0, SPI_CS_LED0 to LED_SPI_CS0, SPI_MOSI_LED_0 to LED_SPI_MOSI_0
Changed lines of the file:
@@
 $EndDescr
 $Comp
-L CONN_01X01 GND0
+L CONN_01X01 KB_GND0
 U 1 1 582F5B39
 P 1250 1000
-F 0 "GND0" H 1450 1000 50  0000 C CNN
+F 0 "KB_GND0" H 1500 1000 50  0000 C CNN
 F 1 "CONN_01X01" V 1350 1000 50  0001 C CNN
 F 2 "Liberry:TH_0.1_1x2_Jumper" H 1250 1000 50  0001 C CNN
@@
 $EndComp
 $Comp
-L CONN_01X01 SDA0
+L CONN_01X01 KB_SDA0
 U 1 1 582FA982
 P 1200 3350
-F 0 "SDA0" H 1550 3350 50  0000 R CNN
+F 0 "KB_SDA0" H 1600 3350 50  0000 R CNN
 F 1 "CONN_01X01" V 1300 3350 50  0001 C CNN
 F 2 "Liberry:TH_0.1_1x2_Jumper" H 1200 3350 50  0001 C CNN
@@
 $EndComp
 $Comp
-L CONN_01X01 SCL0
+L CONN_01X01 KB_SCL0
 U 1 1 583371F2
 P 1200 4050
-F 0 "SCL0" H 1550 4050 50  0000 R CNN
+F 0 "KB_SCL0" H 1600 4050 50  0000 R CNN
 F 1 "CONN_01X01" V 1300 4050 50  0001 C CNN
 F 2 "Liberry:TH_0.1_1x2_Jumper" H 1200 4050 50  0001 C CNN
@@
 $EndComp
 $Comp
-L CONN_01X01 IRQ0
+L CONN_01X01 KB_IRQ0
 U 1 1 58337929
 P 1200 4600
-F 0 "IRQ0" H 1550 4600 50  0000 R CNN
+F 0 "KB_IRQ0" H 1600 4600 50  0000 R CNN
 F 1 "CONN_01X01" V 1300 4600 50  0001 C CNN
 F 2 "Liberry:TH_0.1_1x2_Jumper" H 1200 4600 50  0001 C CNN
@@
 KB_IRQ
 $Comp
-L CONN_01X01 +3.3V0
+L CONN_01X01 KB_+3.3V0
 U 1 1 5833FCAD
 P 1250 800
-F 0 "+3.3V0" H 1500 800 50  0000 C CNN
+F 0 "KB_+3.3V0" H 1550 800 50  0000 C CNN
 F 1 "CONN_01X01" V 1350 800 50  0001 C CNN
 F 2 "Liberry:TH_0.1_1x2_Jumper" H 1250 800 50  0001 C CNN
@@
 $EndComp
 $Comp
-L CONN_01X01 A0
+L CONN_01X01 KB_A0
 U 1 1 588F39C7
 P 1200 5100
-F 0 "A0" H 1550 5100 50  0000 R CNN
+F 0 "KB_A0" H 1550 5100 50  0000 R CNN
 F 1 "CONN_01X01" V 1300 5100 50  0001 C CNN
 F 2 "Liberry:TH_0.1_1x2_Jumper" H 1200 5100 50  0001 C CNN
@@
 $EndComp
 $Comp
-L CONN_01X01 A1
+L CONN_01X01 KB_A1
 U 1 1 588F3BC4
 P 1200 5250
-F 0 "A1" H 1550 5250 50  0000 R CNN
+F 0 "KB_A1" H 1550 5250 50  0000 R CNN
 F 1 "CONN_01X01" V 1300 5250 50  0001 C CNN
 F 2 "Liberry:TH_0.1_1x2_Jumper" H 1200 5250 50  0001 C CNN
@@
 $EndComp
 $Comp
-L CONN_01X01 A2
+L CONN_01X01 KB_A2
 U 1 1 588F3E53
 P 1200 5400
-F 0 "A2" H 1550 5400 50  0000 R CNN
+F 0 "KB_A2" H 1550 5400 50  0000 R CNN
 F 1 "CONN_01X01" V 1300 5400 50  0001 C CNN
 F 2 "Liberry:TH_0.1_1x2_Jumper" H 1200 5400 50  0001 C CNN
@@
 $EndComp
 $Comp
-L CONN_01X01 A3
+L CONN_01X01 KB_A3
 U 1 1 588F404A
 P 1200 5550
-F 0 "A3" H 1550 5550 50  0000 R CNN
+F 0 "KB_A3" H 1550 5550 50  0000 R CNN
 F 1 "CONN_01X01" V 1300 5550 50  0001 C CNN
 F 2 "Liberry:TH_0.1_1x2_Jumper" H 1200 5550 50  0001 C CNN
@@
 $EndComp
 $Comp
-L CONN_01X01 A4
+L CONN_01X01 KB_A4
 U 1 1 588F4154
 P 1200 5700
-F 0 "A4" H 1550 5700 50  0000 R CNN
+F 0 "KB_A4" H 1550 5700 50  0000 R CNN
 F 1 "CONN_01X01" V 1300 5700 50  0001 C CNN
 F 2 "Liberry:TH_0.1_1x2_Jumper" H 1200 5700 50  0001 C CNN
@@
 $EndComp
 $Comp
-L CONN_01X01 A5
+L CONN_01X01 KB_A5
 U 1 1 588F4263
 P 1200 5850
-F 0 "A5" H 1550 5850 50  0000 R CNN
+F 0 "KB_A5" H 1550 5850 50  0000 R CNN
 F 1 "CONN_01X01" V 1300 5850 50  0001 C CNN
 F 2 "Liberry:TH_0.1_1x2_Jumper" H 1200 5850 50  0001 C CNN
@@
 Connection ~ 10250 3350
 $Comp
-L CONN_01X01 GND_LED0
+L CONN_01X01 LED_GND0
 U 1 1 58DF269F
 P 4300 6150
-F 0 "GND_LED0" H 4750 6150 50  0000 R CNN
+F 0 "LED_GND0" H 4750 6150 50  0000 R CNN
 F 1 "CONN_01X01" V 4400 6150 50  0001 C CNN
 F 2 "Liberry:TH_0.1_1x2_Jumper" H 4300 6150 50  0001 C CNN
@@
 $EndComp
 $Comp
-L CONN_01X01 SPI_CLK_LED0
+L CONN_01X01 LED_SPI_CLK0
 U 1 1 58DF2920
 P 4300 5950
-F 0 "SPI_CLK_LED0" H 4900 5950 50  0000 R CNN
+F 0 "LED_SPI_CLK0" H 4900 5950 50  0000 R CNN
 F 1 "CONN_01X01" V 4400 5950 50  0001 C CNN
 F 2 "Liberry:TH_0.1_1x2_Jumper" H 4300 5950 50  0001 C CNN
@@
 $EndComp
 $Comp
-L CONN_01X01 SPI_MOSI_LED_0
+L CONN_01X01 LED_SPI_MOSI_0
 U 1 1 58DF2AA1
 P 4300 5550
-F 0 "SPI_MOSI_LED_0" H 5000 5550 50  0000 R CNN
+F 0 "LED_SPI_MOSI_0" H 5000 5550 50  0000 R CNN
 F 1 "CONN_01X01" V 4400 5550 50  0001 C CNN
 F 2 "Liberry:TH_0.1_1x2_Jumper" H 4300 5550 50  0001 C CNN
@@
 $EndComp
 $Comp
-L CONN_01X01 +3.3V_LED0
+L CONN_01X01 LED_+3.3V0
 U 1 1 58DF2AF2
 P 4300 5350
-F 0 "+3.3V_LED0" H 4850 5350 50  0000 R CNN
+F 0 "LED_+3.3V0" H 4850 5350 50  0000 R CNN
 F 1 "CONN_01X01" V 4400 5350 50  0001 C CNN
 F 2 "Liberry:TH_0.1_1x2_Jumper" H 4300 5350 50  0001 C CNN
@@
 Believotron Wanderlust Beta 1 to Axoloti Core v1.1 translator board
 $Comp
-L CONN_01X01 SPI_CS_LED0
+L CONN_01X01 LED_SPI_CS0
 U 1 1 58E01195
 P 4300 5750
-F 0 "SPI_CS_LED0" H 4850 5750 50  0000 R CNN
+F 0 "LED_SPI_CS0" H 4850 5750 50  0000 R CNN
 F 1 "CONN_01X01" V 4400 5750 50  0001 C CNN
 F 2 "Liberry:TH_0.1_1x2_Jumper" H 4300 5750 50  0001 C CNN
