File: Beta1/PCB1004_Wanderlust_Axoloti_Translator/PCB1004_Wanderlust_Axoloti_Translator.kicad_pcb (KiCad board)
At the start: 2 copper layers, 199 x 64 mm, 102 parts, among them U1 CPT112S, U100 CPT112S, U200 CPT112S

Commit message: Rough placement complete
Parts:
- removed +3.3V0, A0, A1, A2, A3, A4, A5, GND0, IRQ0, SCL0, SDA0: CONN_01X01, Liberry:TH_0.1_1x2_Jumper
- removed C1, C101, C201: 0.1uf, Capacitors_SMD:C_0603
- removed C102, C2, C202: 4.7 uF, Capacitors_SMD:C_0603
- removed CFG_CLK_U1, CFG_CLK_U100, CFG_CLK_U200, CFG_DAT_U1, CFG_DAT_U100, CFG_DAT_U200, GND_U1, GND_U100, GND_U200, PD0, PD1, PD100, PD101, PD102, PD103, PD2, PD3: CONN_01X01, Liberry:single_0.1
- removed G***: LOGO, Liberry:Adventure_Icons_8x2_160x40
- removed PAD0, PAD1, PAD100, PAD101, PAD102, PAD103, PAD104, PAD105, PAD106, PAD107, PAD2, PAD3, PAD4, PAD5, PAD6, PAD7: TOUCHPAD_10CM, Liberry:TOUCH_PAD_10CM
- removed REF** (x2): Fiducial_1mm_Dia_2.54mm_Outer_CopperBottom, Fiducials:Fiducial_1mm_Dia_2.54mm_Outer_CopperBottom
- removed REF** (x6): 1pin, Connect:1pin
- removed TP0, TP1, TP10, TP100, TP101, TP102, TP103, TP104, TP105, TP106, TP107, TP108, TP109, TP11, TP110, TP111, TP2, TP200, TP201, TP202, TP203, TP204, TP205, TP206, TP207, TP208, TP209, TP210, TP211, TP3, TP4, TP5, TP6, TP7, TP8, TP9: CONN_01X01, Liberry:TESTPAD
- removed U1, U100, U200: CPT112S, Liberry:SOIC-24_0.635_1.5x5.2
- removed UKEY0: KEYBOARD_1OCT, Liberry:Keyboard_1_Octave_20CM_V2
- added J1: Axoloti_40Pin, Liberry:Axoloti-40x3, F.Cu at (76.2, -45.5)
- added KB_+3.3V0: CONN_01X01, Liberry:TH_0.1_1x2_Jumper, F.Cu at (26.7, -38.1)
- added KB_A0: CONN_01X01, Liberry:TH_0.1_1x2_Jumper, F.Cu at (39.4, -38.1)
- added KB_A1: CONN_01X01, Liberry:TH_0.1_1x2_Jumper, F.Cu at (41.9, -38.1)
- added KB_A2: CONN_01X01, Liberry:TH_0.1_1x2_Jumper, F.Cu at (44.5, -38.1)
- added KB_A3: CONN_01X01, Liberry:TH_0.1_1x2_Jumper, F.Cu at (47.0, -38.1)
- added KB_A4: CONN_01X01, Liberry:TH_0.1_1x2_Jumper, F.Cu at (49.5, -38.1)
- added KB_A5: CONN_01X01, Liberry:TH_0.1_1x2_Jumper, F.Cu at (52.1, -38.1)
- added KB_GND0: CONN_01X01, Liberry:TH_0.1_1x2_Jumper, F.Cu at (29.2, -38.1)
- added KB_IRQ0: CONN_01X01, Liberry:TH_0.1_1x2_Jumper, F.Cu at (36.8, -38.1)
- added KB_SCL0: CONN_01X01, Liberry:TH_0.1_1x2_Jumper, F.Cu at (34.3, -38.1)
- added KB_SDA0: CONN_01X01, Liberry:TH_0.1_1x2_Jumper, F.Cu at (31.8, -38.1)
- added KNOB_+3.3V0: CONN_01X01, Liberry:TH_0.1_1x2_Jumper, F.Cu at (97.8, -40.6)
- added KNOB_ANALOG_OUT0: CONN_01X01, Liberry:TH_0.1_1x2_Jumper, F.Cu at (102.9, -40.6)
- added KNOB_GND0: CONN_01X01, Liberry:TH_0.1_1x2_Jumper, F.Cu at (82.5, -40.6)
- added KNOB_JOY_SW0: CONN_01X01, Liberry:TH_0.1_1x2_Jumper, F.Cu at (74.9, -40.6)
- added KNOB_JOY_X0: CONN_01X01, Liberry:TH_0.1_1x2_Jumper, F.Cu at (77.5, -40.6)
- added KNOB_JOY_Y0: CONN_01X01, Liberry:TH_0.1_1x2_Jumper, F.Cu at (80.0, -40.6)
- added KNOB_SPI_CLK0: CONN_01X01, Liberry:TH_0.1_1x2_Jumper, F.Cu at (85.1, -40.6)
- added KNOB_SPI_CS_0_7: CONN_01X01, Liberry:TH_0.1_1x2_Jumper, F.Cu at (95.2, -40.6)
- added KNOB_SPI_CS_8_15: CONN_01X01, Liberry:TH_0.1_1x2_Jumper, F.Cu at (92.7, -40.6)
- added KNOB_SPI_MISO0: CONN_01X01, Liberry:TH_0.1_1x2_Jumper, F.Cu at (87.6, -40.6)
- added KNOB_SPI_MOSI0: CONN_01X01, Liberry:TH_0.1_1x2_Jumper, F.Cu at (90.2, -40.6)
- added KNOB_VOL0: CONN_01X01, Liberry:TH_0.1_1x2_Jumper, F.Cu at (100.3, -40.6)
- added LED_+3.3V0: CONN_01X01, Liberry:TH_0.1_1x2_Jumper, F.Cu at (57.1, -38.1)
- added LED_GND0: CONN_01X01, Liberry:TH_0.1_1x2_Jumper, F.Cu at (67.3, -38.1)
- added LED_SPI_CLK0: CONN_01X01, Liberry:TH_0.1_1x2_Jumper, F.Cu at (64.8, -38.1)
- added LED_SPI_CS0: CONN_01X01, Liberry:TH_0.1_1x2_Jumper, F.Cu at (62.2, -38.1)
- added LED_SPI_MOSI_0: CONN_01X01, Liberry:TH_0.1_1x2_Jumper, F.Cu at (59.7, -38.1)
- R301, R302, R303: moved to F.Cu
- moved R303 28.2 mm to (38.9, -43.2)
- moved R301 26.4 mm to (36.1, -43.2), turned to 0 degrees
- moved R302 24.8 mm to (33.0, -43.2), turned to 0 degrees
Connections:
- net +3V3 renamed /VCC_A
- R301 pad 2: /SDA -> /I2C_SDA
- R302 pad 2: /SCL -> /I2C_SCL
- R303 pad 2: /IRQ -> /KB_IRQ
Routing:
- net GND: track 9574.6 -> 0.00 mm, vias 23 -> 0
- net (no net): track 1033.8 -> 0.00 mm, vias 3 -> 0
- net /CHIP_04: track 162.0 -> 0.00 mm, vias 1 -> 0
- net /CHIP_104: track 162.0 -> 0.00 mm, vias 1 -> 0
- net /CHIP_111: track 155.7 -> 0.00 mm, vias 1 -> 0
- net /CHIP_206: track 154.7 -> 0.00 mm, vias 1 -> 0
- net /CHIP_211: track 146.2 -> 0.00 mm, vias 1 -> 0
- net /CHIP_11: track 135.8 -> 0.00 mm, vias 1 -> 0
- net /CHIP_205: track 131.1 -> 0.00 mm, vias 1 -> 0
- net /CHIP_210: track 123.0 -> 0.00 mm, vias 1 -> 0
- net /CHIP_105: track 122.8 -> 0.00 mm, vias 1 -> 0
- net /CHIP_05: track 120.7 -> 0.00 mm, vias 1 -> 0
- net /CHIP_110: track 110.5 -> 0.00 mm, vias 1 -> 0
- net /SCL: track 108.1 -> 0.00 mm, vias 2 -> 0
- net /CHIP_204: track 107.4 -> 0.00 mm, vias 1 -> 0
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Other:
- board text removed: "+3.3V"
- board text removed: "0.1uF"
- board text removed: "10K x3"
- board text removed: "4.7uF"
- board text removed: "A0"
- board text removed: "A1"
- board text removed: "A2"
- board text removed: "A3"
- board text removed: "A4"
- board text removed: "A5"
- board text removed: "CPT112S-A02-GU"
- board text removed: "GND"
- board text removed: "IRQ"
- board text removed: "Open Source License at: https://github.com/Believotron/BelievotronWanderlustHardware Marketing pap: believotron.com The good stuff: http://community.believotron.com/"
- board text removed: "Open source MIT license files at: github.com/Believotron/BelievotronWanderlustHardware Replacement parts, upgrades, updates, new gear, and marketing pap: Believotron.com For help, bug reporting, dev-blogs, or joy at your bonkers-cool creation, the good stuff is here: community.believotron.com"
- board text removed: "PCB1003_1OCTAVE_16PAD_Alt_2017-03-31 Beta-1 Believotron Wanderlust 1/2 H Keypad 1 Octave Piano, 16 Pads 6CH Analog Mezzanine Expansion headers"
- board text removed: "SCL"
- board text removed: "SDA"
- board text removed: "TP show which bit each pad is. Example: TP4 is Bit 4. TP211 is chip 200, bit 11"

Commit message: Created PCB files. Ready for fab.
Parts:
- moved KNOB_ANALOG_OUT0 5.08 mm to (108.0, -40.6)
Routing:
- net GND: track 0.00 -> 159.4 mm
- net /KNOB_CS_8_15: track 0.00 -> 96.3 mm
- net /KNOB_CS_0_7: track 0.00 -> 93.4 mm
- net /JOY_X: track 0.00 -> 80.9 mm
- net /KB_IRQ: track 0.00 -> 78.6 mm
- net /JOY_Y: track 0.00 -> 69.2 mm
- net /VOLUME: track 0.00 -> 62.0 mm, vias 0 -> 1
- net /VCC_B: track 0.00 -> 55.0 mm
- net /VCC_A: track 0.00 -> 54.0 mm
- net /ANALOG_OUT: track 0.00 -> 49.3 mm
- net /SPI_MOSI: track 0.00 -> 48.0 mm
- net /SPI_CLK: track 0.00 -> 37.4 mm
- net /KB_A5: track 0.00 -> 29.9 mm
- net /KB_A4: track 0.00 -> 29.9 mm
- net /KB_A3: track 0.00 -> 27.4 mm
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Other:
- board size 199 x 64 mm -> 111.8 x 27.9 mm
- board text added: "Analog out"
- board text added: "KB0"
- board text added: "KNOB0"
- board text added: "LED0"
- board text added: "PCB1004_Wanderlust_Axoloti_Translator_2017-03-31 Beta1 Open source MIT license files at: github.com/Believotron/BelievotronWanderlustHardware Replacement parts, upgrades, updates, new gear, and marketing pap: Believotron.com For help, bug reporting, dev-blogs, or joy at your bonkers-cool creation, the good stuff is here: community.believotron.com"
