File: Beta1/PCB1005_KnobCore/_saved_PCB1005-KnobCore.sch (KiCad schematic (older format))
At the start: 34 parts, among them J1 Axoloti_40Pin, U10 OLED_128x32_I2C, U1000 MCP3008T-I/SL, U2 MCP3008T-I/SL, U20 OLED_128x32_I2C, U30 OLED_128x32_I2C, U5 I2C_1x4MUX_TCA9546A

Commit message: Initial Placement
Parts:
- renumbered RV_VOL to RV_VOL1
Changed lines of the file:
@@
 $EndComp
 $Comp
-L GND #PWR01
+L GND #PWR2
 U 1 1 582E602B
 P 2150 1750
-F 0 "#PWR01" H 2150 1500 50  0001 C CNN
+F 0 "#PWR2" H 2150 1500 50  0001 C CNN
 F 1 "GND" H 2150 1600 50  0000 C CNN
 F 2 "" H 2150 1750 50  0000 C CNN
@@
 $EndComp
 $Comp
-L +3.3V #PWR02
+L +3.3V #PWR1
 U 1 1 582E6042
 P 2150 1300
-F 0 "#PWR02" H 2150 1150 50  0001 C CNN
+F 0 "#PWR1" H 2150 1150 50  0001 C CNN
 F 1 "+3.3V" H 2150 1440 50  0000 C CNN
 F 2 "" H 2150 1300 50  0000 C CNN
@@
 $EndComp
 $Comp
-L GND #PWR03
+L GND #PWR6
 U 1 1 582E62D8
 P 2950 1750
-F 0 "#PWR03" H 2950 1500 50  0001 C CNN
+F 0 "#PWR6" H 2950 1500 50  0001 C CNN
 F 1 "GND" H 2950 1600 50  0000 C CNN
 F 2 "" H 2950 1750 50  0000 C CNN
@@
 $EndComp
 $Comp
-L +3.3V #PWR04
+L +3.3V #PWR5
 U 1 1 582E62DE
 P 2950 1300
-F 0 "#PWR04" H 2950 1150 50  0001 C CNN
+F 0 "#PWR5" H 2950 1150 50  0001 C CNN
 F 1 "+3.3V" H 2950 1440 50  0000 C CNN
 F 2 "" H 2950 1300 50  0000 C CNN
@@
 $EndComp
 $Comp
-L GND #PWR05
+L GND #PWR8
 U 1 1 582E632D
 P 3800 1750
-F 0 "#PWR05" H 3800 1500 50  0001 C CNN
+F 0 "#PWR8" H 3800 1500 50  0001 C CNN
 F 1 "GND" H 3800 1600 50  0000 C CNN
 F 2 "" H 3800 1750 50  0000 C CNN
@@
 $EndComp
 $Comp
-L +3.3V #PWR06
+L +3.3V #PWR7
 U 1 1 582E6333
 P 3800 1300
-F 0 "#PWR06" H 3800 1150 50  0001 C CNN
+F 0 "#PWR7" H 3800 1150 50  0001 C CNN
 F 1 "+3.3V" H 3800 1440 50  0000 C CNN
 F 2 "" H 3800 1300 50  0000 C CNN
@@
 $EndComp
 $Comp
-L GND #PWR07
+L GND #PWR12
 U 1 1 582E6345
 P 4600 1750
-F 0 "#PWR07" H 4600 1500 50  0001 C CNN
+F 0 "#PWR12" H 4600 1500 50  0001 C CNN
 F 1 "GND" H 4600 1600 50  0000 C CNN
 F 2 "" H 4600 1750 50  0000 C CNN
@@
 $EndComp
 $Comp
-L +3.3V #PWR08
+L +3.3V #PWR11
 U 1 1 582E634B
 P 4600 1300
-F 0 "#PWR08" H 4600 1150 50  0001 C CNN
+F 0 "#PWR11" H 4600 1150 50  0001 C CNN
 F 1 "+3.3V" H 4600 1440 50  0000 C CNN
 F 2 "" H 4600 1300 50  0000 C CNN
@@
 $EndComp
 $Comp
-L GND #PWR09
+L GND #PWR14
 U 1 1 582E665F
 P 5500 1750
-F 0 "#PWR09" H 5500 1500 50  0001 C CNN
+F 0 "#PWR14" H 5500 1500 50  0001 C CNN
 F 1 "GND" H 5500 1600 50  0000 C CNN
 F 2 "" H 5500 1750 50  0000 C CNN
@@
 $EndComp
 $Comp
-L +3.3V #PWR010
+L +3.3V #PWR13
 U 1 1 582E6665
 P 5500 1300
-F 0 "#PWR010" H 5500 1150 50  0001 C CNN
+F 0 "#PWR13" H 5500 1150 50  0001 C CNN
 F 1 "+3.3V" H 5500 1440 50  0000 C CNN
 F 2 "" H 5500 1300 50  0000 C CNN
@@
 $EndComp
 $Comp
-L GND #PWR011
+L GND #PWR16
 U 1 1 582E6677
 P 6300 1750
-F 0 "#PWR011" H 6300 1500 50  0001 C CNN
+F 0 "#PWR16" H 6300 1500 50  0001 C CNN
 F 1 "GND" H 6300 1600 50  0000 C CNN
 F 2 "" H 6300 1750 50  0000 C CNN
@@
 $EndComp
 $Comp
-L +3.3V #PWR012
+L +3.3V #PWR15
 U 1 1 582E667D
 P 6300 1300
-F 0 "#PWR012" H 6300 1150 50  0001 C CNN
+F 0 "#PWR15" H 6300 1150 50  0001 C CNN
 F 1 "+3.3V" H 6300 1440 50  0000 C CNN
 F 2 "" H 6300 1300 50  0000 C CNN
@@
 $EndComp
 $Comp
-L GND #PWR013
+L GND #PWR20
 U 1 1 582E668F
 P 7150 1750
-F 0 "#PWR013" H 7150 1500 50  0001 C CNN
+F 0 "#PWR20" H 7150 1500 50  0001 C CNN
 F 1 "GND" H 7150 1600 50  0000 C CNN
 F 2 "" H 7150 1750 50  0000 C CNN
@@
 $EndComp
 $Comp
-L +3.3V #PWR014
+L +3.3V #PWR19
 U 1 1 582E6695
 P 7150 1300
-F 0 "#PWR014" H 7150 1150 50  0001 C CNN
+F 0 "#PWR19" H 7150 1150 50  0001 C CNN
 F 1 "+3.3V" H 7150 1440 50  0000 C CNN
 F 2 "" H 7150 1300 50  0000 C CNN
@@
 $EndComp
 $Comp
-L GND #PWR015
+L GND #PWR22
 U 1 1 582E66A7
 P 7950 1750
-F 0 "#PWR015" H 7950 1500 50  0001 C CNN
+F 0 "#PWR22" H 7950 1500 50  0001 C CNN
 F 1 "GND" H 7950 1600 50  0000 C CNN
 F 2 "" H 7950 1750 50  0000 C CNN
@@
 $EndComp
 $Comp
-L +3.3V #PWR016
+L +3.3V #PWR21
 U 1 1 582E66AD
 P 7950 1300
-F 0 "#PWR016" H 7950 1150 50  0001 C CNN
+F 0 "#PWR21" H 7950 1150 50  0001 C CNN
 F 1 "+3.3V" H 7950 1440 50  0000 C CNN
 F 2 "" H 7950 1300 50  0000 C CNN
@@
 $EndComp
 $Comp
-L GND #PWR017
+L GND #PWR26
 U 1 1 582E3FD0
 P 9000 1450
-F 0 "#PWR017" H 9000 1200 50  0001 C CNN
+F 0 "#PWR26" H 9000 1200 50  0001 C CNN
 F 1 "GND" H 9000 1300 50  0000 C CNN
 F 2 "" H 9000 1450 50  0000 C CNN
@@
 $EndComp
 $Comp
-L +3.3V #PWR018
+L +3.3V #PWR25
 U 1 1 582E424D
 P 9000 750
-F 0 "#PWR018" H 9000 600 50  0001 C CNN
+F 0 "#PWR25" H 9000 600 50  0001 C CNN
 F 1 "+3.3V" H 9000 890 50  0000 C CNN
 F 2 "" H 9000 750 50  0000 C CNN
@@
 P0
 $Comp
-L GND #PWR019
+L GND #PWR30
 U 1 1 582E4C7F
 P 11350 2950
-F 0 "#PWR019" H 11350 2700 50  0001 C CNN
+F 0 "#PWR30" H 11350 2700 50  0001 C CNN
 F 1 "GND" H 11350 2800 50  0000 C CNN
 F 2 "" H 11350 2950 50  0000 C CNN
@@
 $EndComp
 $Comp
-L GND #PWR036
+L GND #PWR24
 U 1 1 582F416B
 P 8950 4000
-F 0 "#PWR036" H 8950 3750 50  0001 C CNN
+F 0 "#PWR24" H 8950 3750 50  0001 C CNN
 F 1 "GND" H 8950 3850 50  0000 C CNN
 F 2 "" H 8950 4000 50  0000 C CNN
@@
 $EndComp
 $Comp
-L +3.3V #PWR037
+L +3.3V #PWR23
 U 1 1 582F4171
 P 8950 3500
-F 0 "#PWR037" H 8950 3350 50  0001 C CNN
+F 0 "#PWR23" H 8950 3350 50  0001 C CNN
 F 1 "+3.3V" H 8950 3640 50  0000 C CNN
 F 2 "" H 8950 3500 50  0000 C CNN
@@
 JOY_0_0
 $Comp
-L GND #PWR038
+L GND #PWR29
 U 1 1 582F4178
 P 11300 5700
-F 0 "#PWR038" H 11300 5450 50  0001 C CNN
+F 0 "#PWR29" H 11300 5450 50  0001 C CNN
 F 1 "GND" H 11300 5550 50  0000 C CNN
 F 2 "" H 11300 5700 50  0000 C CNN
@@
 $EndComp
 $Comp
-L +3.3V #PWR039
+L +3.3V #PWR9
 U 1 1 5880F86D
 P 3900 8650
-F 0 "#PWR039" H 3900 8500 50  0001 C CNN
+F 0 "#PWR9" H 3900 8500 50  0001 C CNN
 F 1 "+3.3V" H 3900 8790 50  0000 C CNN
 F 2 "" H 3900 8650 50  0000 C CNN
@@
 $EndComp
 $Comp
-L GND #PWR040
+L GND #PWR10
 U 1 1 5880F8DB
 P 4000 10100
-F 0 "#PWR040" H 4000 9850 50  0001 C CNN
+F 0 "#PWR10" H 4000 9850 50  0001 C CNN
 F 1 "GND" H 4000 9950 50  0000 C CNN
 F 2 "" H 4000 10100 50  0000 C CNN
@@
 I2C_SDA
 $Comp
-L GND #PWR043
+L GND #PWR34
 U 1 1 591BA513
 P 14900 6300
-F 0 "#PWR043" H 14900 6050 50  0001 C CNN
+F 0 "#PWR34" H 14900 6050 50  0001 C CNN
 F 1 "GND" H 14900 6150 50  0000 C CNN
 F 2 "" H 14900 6300 50  0000 C CNN
@@
 $EndComp
 $Comp
-L +3.3V #PWR044
+L +3.3V #PWR33
 U 1 1 591E099F
 P 14900 1950
-F 0 "#PWR044" H 14900 1800 50  0001 C CNN
+F 0 "#PWR33" H 14900 1800 50  0001 C CNN
 F 1 "+3.3V" H 14900 2090 50  0000 C CNN
 F 2 "" H 14900 1950 50  0000 C CNN
@@
 $EndComp
 $Comp
-L +3.3V #PWR045
+L +3.3V #PWR38
 U 1 1 591E1B3B
 P 22200 1800
-F 0 "#PWR045" H 22200 1650 50  0001 C CNN
+F 0 "#PWR38" H 22200 1650 50  0001 C CNN
 F 1 "+3.3V" H 22200 1940 50  0000 C CNN
 F 2 "" H 22200 1800 50  0000 C CNN
@@
 I2C_SCL3
 $Comp
-L GND #PWR046
+L GND #PWR37
 U 1 1 591E1666
 P 20900 3850
-F 0 "#PWR046" H 20900 3600 50  0001 C CNN
+F 0 "#PWR37" H 20900 3600 50  0001 C CNN
 F 1 "GND" H 20900 3700 50  0000 C CNN
 F 2 "" H 20900 3850 50  0000 C CNN
@@
 $EndComp
 $Comp
-L GND #PWR047
+L GND #PWR36
 U 1 1 591E16DA
 P 20400 2200
-F 0 "#PWR047" H 20400 1950 50  0001 C CNN
+F 0 "#PWR36" H 20400 1950 50  0001 C CNN
 F 1 "GND" H 20400 2050 50  0000 C CNN
 F 2 "" H 20400 2200 50  0000 C CNN
@@
 $EndComp
 $Comp
-L +3.3V #PWR048
+L +3.3V #PWR35
 U 1 1 591E5102
 P 20400 1550
-F 0 "#PWR048" H 20400 1400 50  0001 C CNN
+F 0 "#PWR35" H 20400 1400 50  0001 C CNN
 F 1 "+3.3V" H 20400 1690 50  0000 C CNN
 F 2 "" H 20400 1550 50  0000 C CNN
@@
 Connection ~ 14650 4100
 $Comp
-L +3.3V #PWR049
+L +3.3V #PWR39
 U 1 1 591F153F
 P 26450 1650
-F 0 "#PWR049" H 26450 1500 50  0001 C CNN
+F 0 "#PWR39" H 26450 1500 50  0001 C CNN
 F 1 "+3.3V" H 26450 1790 50  0000 C CNN
 F 2 "" H 26450 1650 50  0000 C CNN
@@
 Connection ~ 26450 2950
 $Comp
-L GND #PWR050
+L GND #PWR40
 U 1 1 591F1D12
 P 26650 4400
-F 0 "#PWR050" H 26650 4150 50  0001 C CNN
+F 0 "#PWR40" H 26650 4150 50  0001 C CNN
 F 1 "GND" H 26650 4250 50  0000 C CNN
 F 2 "" H 26650 4400 50  0000 C CNN
@@
 $EndComp
 $Comp
-L +3.3V #PWR?
+L +3.3V #PWR17
 U 1 1 592E37F7
 P 6700 8650
-F 0 "#PWR?" H 6700 8500 50  0001 C CNN
+F 0 "#PWR17" H 6700 8500 50  0001 C CNN
 F 1 "+3.3V" H 6700 8790 50  0000 C CNN
 F 2 "" H 6700 8650 50  0000 C CNN
@@
 $EndComp
 $Comp
-L GND #PWR?
+L GND #PWR18
 U 1 1 592E37FD
 P 6800 10100
-F 0 "#PWR?" H 6800 9850 50  0001 C CNN
+F 0 "#PWR18" H 6800 9850 50  0001 C CNN
 F 1 "GND" H 6800 9950 50  0000 C CNN
 F 2 "" H 6800 10100 50  0000 C CNN
@@
 $EndComp
 $Comp
-L +3.3V #PWR?
+L +3.3V #PWR27
 U 1 1 592E39C6
 P 9500 8650
-F 0 "#PWR?" H 9500 8500 50  0001 C CNN
+F 0 "#PWR27" H 9500 8500 50  0001 C CNN
 F 1 "+3.3V" H 9500 8790 50  0000 C CNN
 F 2 "" H 9500 8650 50  0000 C CNN
@@
 $EndComp
 $Comp
-L GND #PWR?
+L GND #PWR28
 U 1 1 592E39CC
 P 9600 10100
-F 0 "#PWR?" H 9600 9850 50  0001 C CNN
+F 0 "#PWR28" H 9600 9850 50  0001 C CNN
 F 1 "GND" H 9600 9950 50  0000 C CNN
 F 2 "" H 9600 10100 50  0000 C CNN
@@
 $EndComp
 $Comp
-L +3.3V #PWR?
+L +3.3V #PWR31
 U 1 1 592E39E8
 P 12300 8650
-F 0 "#PWR?" H 12300 8500 50  0001 C CNN
+F 0 "#PWR31" H 12300 8500 50  0001 C CNN
 F 1 "+3.3V" H 12300 8790 50  0000 C CNN
 F 2 "" H 12300 8650 50  0000 C CNN
@@
 $EndComp
 $Comp
-L GND #PWR?
+L GND #PWR32
 U 1 1 592E39EE
 P 12400 10100
-F 0 "#PWR?" H 12400 9850 50  0001 C CNN
+F 0 "#PWR32" H 12400 9850 50  0001 C CNN
 F 1 "GND" H 12400 9950 50  0000 C CNN
 F 2 "" H 12400 10100 50  0000 C CNN
@@
 	15050 3700 15900 3700
 $Comp
-L POT RV_VOL
+L POT RV_VOL1
 U 1 1 592EADD2
 P 2150 3100
-F 0 "RV_VOL" H 2150 2850 50  0000 C CNN
+F 0 "RV_VOL1" H 2150 2850 50  0000 C CNN
 F 1 "POT" H 2150 3100 50  0000 C CNN
 F 2 "Liberry:RV09AF-40-20K-B10K" H 2150 3100 50  0001 C CNN
@@
 $EndComp
 $Comp
-L GND #PWR?
+L GND #PWR4
 U 1 1 592EADD8
 P 2150 3300
-F 0 "#PWR?" H 2150 3050 50  0001 C CNN
+F 0 "#PWR4" H 2150 3050 50  0001 C CNN
 F 1 "GND" H 2150 3150 50  0000 C CNN
 F 2 "" H 2150 3300 50  0000 C CNN
@@
 $EndComp
 $Comp
-L +3.3V #PWR?
+L +3.3V #PWR3
 U 1 1 592EADDE
 P 2150 2850
-F 0 "#PWR?" H 2150 2700 50  0001 C CNN
+F 0 "#PWR3" H 2150 2700 50  0001 C CNN
 F 1 "+3.3V" H 2150 2990 50  0000 C CNN
 F 2 "" H 2150 2850 50  0000 C CNN
