File: Beta1/PCB1006-Fader16/PCB1006-Fader8.sch (KiCad schematic (older format))
At the start: 33 parts, among them U1000 MCP3008T-I/SL, U2 MCP3008T-I/SL

Commit message: Routing complete
Parts:
- removed C2: 0.1u, Capacitors_SMD:C_0603, symbol C
- removed RV10, RV11, RV12, RV13, RV14, RV15, RV8, RV9: POT, Liberry:RV09AF-40-20K-B10K, symbol POT
- removed SPI_CS_8_15: CONN_01X01, Liberry:TH_0.1_1x2_Jumper, symbol CONN_01X01
- removed U2: MCP3008T-I/SL, Liberry:SOIC-16, symbol MCP3008T-I/SL
- RV0, RV1, RV2, RV3, RV4, RV5, RV6, RV7: footprint Liberry:RV09AF-40-20K-B10K -> Liberry:LINEAR_POT_TT_ELECTRONICS_PS45M; MFG Alpha Taiwan -> TT-ELECTRONICS_BI; MPN RV09AF-40-20K-B10K -> PS45M-0MC2BR10K
Connections:
- net labels removed: CS_LED_8_15, P10, P11, P12, P13, P14, P15, P8, P9
- wire segments 113 -> 68
Other:
- note added: "2017-06-09"
- note added: "Believotron Wanderlust PCB 8 CH Analog Fader + JoyXY + Volume"
- note removed: "2017-03-31"
- note removed: "Believotron Wanderlust PCB 16 CH Analog Knob + JoyXY + Volume"
