File: Beta1/PCB1008_Knob8_Vert/PCB1008-Knob8_Vert.sch (KiCad schematic (older format))
At the start: 34 parts, among them J1 Axoloti_40Pin, U10 OLED_128x32_I2C, U1000 MCP3008T-I/SL, U2 MCP3008T-I/SL, U20 OLED_128x32_I2C, U30 OLED_128x32_I2C, U40 OLED_128x32_I2C, U5 I2C_1x4MUX_TCA9546A

Commit message: Converted old sch
Added QTY 2, 1x4 connectors
Changed Pots to 1M long life pot
Removed OLED ckt
Removed Joy ckt
Parts:
- removed C1, C2: 0.1u, Capacitors_SMD:C_0603, symbol C
- removed J1: Axoloti_40Pin, Liberry:Axoloti-40x1_slim, symbol Axoloti_40Pin
- removed JOY0, JOY1, JOY2, JOY3: XYJOY_Alps, Liberry:JOY_ALPS_RKJXV1224005, symbol XYJOY_Alps
- removed RC0, RC10, RC20, RC30, RC40, RD0, RD10, RD20, RD30, RD40, RR0: 10K, Resistors_SMD:R_0603, symbol R
- removed U10, U20, U30, U40: OLED_128x32_I2C, Liberry:OLED_128x32, symbol OLED_128x32_I2C
- removed U2: MCP3008T-I/SL, Liberry:SOIC-16, symbol MCP3008T-I/SL
- removed U5: I2C_1x4MUX_TCA9546A, Liberry:SOIC-16_1.27x5.4, symbol I2C_1x4MUX_TCA9546A
- added P0-0, P0-1, P0-2, P0-3, P1-0, P1-1, P1-2, P1-3: CONN_01X01, Liberry:TH_0.1_1x2_Jumper, symbol CONN_01X01
- RV0, RV1, RV2, RV3, RV4, RV5, RV6, RV7: footprint Liberry:RV09AF-40-20K-B10K -> Liberry:POT_ALPS_RK09Y11L0001; MPN RV09AF-40-20K-B10K -> RK09Y11L0001
Connections:
- net labels removed: !OLED_RESET, CS_8_15, I2C_SCL, I2C_SCL0, I2C_SCL1, I2C_SCL2, I2C_SCL3, I2C_SDA, I2C_SDA0, I2C_SDA1, I2C_SDA2, I2C_SDA3, JOY_0_0, JOY_0_1, JOY_0_SW, JOY_1_0, JOY_1_1, JOY_1_SW, JOY_2_0, JOY_2_1, JOY_2_SW, JOY_3_0, JOY_3_1, JOY_3_SW, VOLUME
- wire segments 200 -> 54

Commit message: Finished rough placement and 3D model
Parts:
- removed P0-0, P0-1, P0-2, P0-3, P1-0, P1-1, P1-2, P1-3: CONN_01X01, Liberry:TH_0.1_1x2_Jumper, symbol CONN_01X01
- added J0, J1: CON_1x4, Liberry:CON_0.1x4_SAMTEC_TSW-104-08-L-S-RA, symbol CON_1x4
Other:
- note added: "TSW-104-08-L-S-RA"
Changed lines of the file:
@@
 LIBS:Zilog
 LIBS:believotron_wanderlust
+LIBS:PCB1008-Knob8_Vert-cache
 EELAYER 25 0
 EELAYER END
@@
 Wire Wire Line
 	11200 1750 11850 1750
-$Comp
-L CONN_01X01 P1-0
-U 1 1 597BE2D8
-P 2450 3900
-F 0 "P1-0" H 2550 3900 50  0000 L CNN
-F 1 "CONN_01X01" V 2550 3900 50  0001 C CNN
-F 2 "Liberry:TH_0.1_1x2_Jumper" H 2500 4150 50  0001 C CNN
-F 3 "" H 2450 3900 50  0000 C CNN
-	1    2450 3900
-	-1   0    0    1
-$EndComp
-$Comp
-L CONN_01X01 P1-1
-U 1 1 597BF147
-P 2450 4000
-F 0 "P1-1" H 2550 4000 50  0000 L CNN
-F 1 "CONN_01X01" V 2550 4000 50  0001 C CNN
-F 2 "Liberry:TH_0.1_1x2_Jumper" H 2500 4250 50  0001 C CNN
-F 3 "" H 2450 4000 50  0000 C CNN
-	1    2450 4000
-	-1   0    0    1
-$EndComp
-$Comp
-L CONN_01X01 P1-2
-U 1 1 597BF1CB
-P 2450 4100
-F 0 "P1-2" H 2550 4100 50  0000 L CNN
-F 1 "CONN_01X01" V 2550 4100 50  0001 C CNN
-F 2 "Liberry:TH_0.1_1x2_Jumper" H 2500 4350 50  0001 C CNN
-F 3 "" H 2450 4100 50  0000 C CNN
-	1    2450 4100
-	-1   0    0    1
-$EndComp
-$Comp
-L CONN_01X01 P1-3
-U 1 1 597BF24A
-P 2450 4200
-F 0 "P1-3" H 2550 4200 50  0000 L CNN
-F 1 "CONN_01X01" V 2550 4200 50  0001 C CNN
-F 2 "Liberry:TH_0.1_1x2_Jumper" H 2500 4450 50  0001 C CNN
-F 3 "" H 2450 4200 50  0000 C CNN
-	1    2450 4200
-	-1   0    0    1
-$EndComp
-$Comp
-L CONN_01X01 P0-0
-U 1 1 597BF856
-P 2450 3150
-F 0 "P0-0" H 2550 3150 50  0000 L CNN
-F 1 "CONN_01X01" V 2550 3150 50  0001 C CNN
-F 2 "Liberry:TH_0.1_1x2_Jumper" H 2500 3400 50  0001 C CNN
-F 3 "" H 2450 3150 50  0000 C CNN
-	1    2450 3150
-	-1   0    0    1
-$EndComp
-$Comp
-L CONN_01X01 P0-1
-U 1 1 597BF85D
-P 2450 3250
-F 0 "P0-1" H 2550 3250 50  0000 L CNN
-F 1 "CONN_01X01" V 2550 3250 50  0001 C CNN
-F 2 "Liberry:TH_0.1_1x2_Jumper" H 2500 3500 50  0001 C CNN
-F 3 "" H 2450 3250 50  0000 C CNN
-	1    2450 3250
-	-1   0    0    1
-$EndComp
-$Comp
-L CONN_01X01 P0-2
-U 1 1 597BF864
-P 2450 3350
-F 0 "P0-2" H 2550 3350 50  0000 L CNN
-F 1 "CONN_01X01" V 2550 3350 50  0001 C CNN
-F 2 "Liberry:TH_0.1_1x2_Jumper" H 2500 3600 50  0001 C CNN
-F 3 "" H 2450 3350 50  0000 C CNN
-	1    2450 3350
-	-1   0    0    1
-$EndComp
-$Comp
-L CONN_01X01 P0-3
-U 1 1 597BF86B
-P 2450 3450
-F 0 "P0-3" H 2550 3450 50  0000 L CNN
-F 1 "CONN_01X01" V 2550 3450 50  0001 C CNN
-F 2 "Liberry:TH_0.1_1x2_Jumper" H 2500 3700 50  0001 C CNN
-F 3 "" H 2450 3450 50  0000 C CNN
-	1    2450 3450
-	-1   0    0    1
-$EndComp
-Wire Wire Line
-	2650 3150 3700 3150
-Wire Wire Line
-	2650 3250 3700 3250
-Wire Wire Line
-	2650 3350 3700 3350
-Wire Wire Line
-	2650 3450 4050 3450
-Wire Wire Line
-	2650 3900 3700 3900
-Wire Wire Line
-	2650 4000 3700 4000
-Wire Wire Line
-	2650 4100 4050 4100
-Wire Wire Line
-	2650 4200 4050 4200
+Wire Wire Line
+	2500 3000 3550 3000
+Wire Wire Line
+	2500 3150 3550 3150
+Wire Wire Line
+	2500 3300 3550 3300
+Wire Wire Line
+	2500 3450 4050 3450
+Wire Wire Line
+	2500 4050 3550 4050
+Wire Wire Line
+	2500 4200 3550 4200
+Wire Wire Line
+	2500 4500 4050 4500
 $Comp
 L GND #PWR?
 U 1 1 597C19D1
-P 4050 4400
-F 0 "#PWR?" H 4050 4150 50  0001 C CNN
-F 1 "GND" H 4050 4250 50  0000 C CNN
-F 2 "" H 4050 4400 50  0000 C CNN
-F 3 "" H 4050 4400 50  0000 C CNN
-	1    4050 4400
-	1    0    0    -1
-$EndComp
-Wire Wire Line
-	4050 3450 4050 4400
-Connection ~ 4050 4200
-Text Label 2750 3150 0    60   ~ 0
+P 4050 4700
+F 0 "#PWR?" H 4050 4450 50  0001 C CNN
+F 1 "GND" H 4050 4550 50  0000 C CNN
+F 2 "" H 4050 4700 50  0000 C CNN
+F 3 "" H 4050 4700 50  0000 C CNN
+	1    4050 4700
+	1    0    0    -1
+$EndComp
+Wire Wire Line
+	4050 3450 4050 4700
+Connection ~ 4050 4500
+Text Label 2600 3000 0    60   ~ 0
 SPI_CLK
-Text Label 2750 3250 0    60   ~ 0
+Text Label 2600 3150 0    60   ~ 0
 SPI_MOSI
-Text Label 2750 3350 0    60   ~ 0
+Text Label 2600 3300 0    60   ~ 0
 SPI_MISO
-Text Label 2750 4000 0    60   ~ 0
+Text Label 2600 4200 0    60   ~ 0
 CS_0_7
 $Comp
 L +3.3V #PWR?
 U 1 1 597C2505
-P 3700 3900
-F 0 "#PWR?" H 3700 3750 50  0001 C CNN
-F 1 "+3.3V" H 3700 4040 50  0000 C CNN
-F 2 "" H 3700 3900 50  0000 C CNN
-F 3 "" H 3700 3900 50  0000 C CNN
-	1    3700 3900
-	1    0    0    -1
-$EndComp
-Connection ~ 4050 4100
+P 3550 4050
+F 0 "#PWR?" H 3550 3900 50  0001 C CNN
+F 1 "+3.3V" H 3550 4190 50  0000 C CNN
+F 2 "" H 3550 4050 50  0000 C CNN
+F 3 "" H 3550 4050 50  0000 C CNN
+	1    3550 4050
+	1    0    0    -1
+$EndComp
+$Comp
+L CON_1x4 J0
+U 1 1 597BBDCE
+P 2300 3000
+F 0 "J0" H 2450 3200 60  0000 C CNN
+F 1 "CON_1x4" H 2400 2400 60  0000 C CNN
+F 2 "Liberry:CON_0.1x4_SAMTEC_TSW-104-08-L-S-RA" H 2300 3000 60  0001 C CNN
+F 3 "" H 2300 3000 60  0001 C CNN
+	1    2300 3000
+	-1   0    0    -1
+$EndComp
+Text Notes 1700 4800 0    60   ~ 0
+TSW-104-08-L-S-RA
+$Comp
+L CON_1x4 J1
+U 1 1 597BC60B
+P 2300 4050
+F 0 "J1" H 2450 4250 60  0000 C CNN
+F 1 "CON_1x4" H 2400 3450 60  0000 C CNN
+F 2 "Liberry:CON_0.1x4_SAMTEC_TSW-104-08-L-S-RA" H 2300 4050 60  0001 C CNN
+F 3 "" H 2300 4050 60  0001 C CNN
+	1    2300 4050
+	-1   0    0    -1
+$EndComp
+Wire Wire Line
+	2500 4350 4050 4350
+Connection ~ 4050 4350
+Text Notes 1700 3750 0    60   ~ 0
+TSW-104-08-L-S-RA
 $EndSCHEMATC
