File: Beta1/PCB1008_Knob8_Vert/PCB1008-Knob8_Vert.kicad_pcb (KiCad board)
At the start: 2 copper layers, 160 x 15.9 mm, 18 parts, among them J0 CON_1x4, J1 CON_1x4, U1000 MCP3008T-I/SL

Commit message: Routing complete
Routing:
- net +3V3: track 0.00 -> 252.2 mm
- net /SPI_MISO: track 0.00 -> 67.8 mm
- net /P0: track 0.00 -> 67.2 mm
- net /P7: track 0.00 -> 66.7 mm
- net /SPI_MOSI: track 0.00 -> 65.1 mm
- net /CS_0_7: track 0.00 -> 63.9 mm
- net /SPI_CLK: track 0.00 -> 59.2 mm
- net /P6: track 0.00 -> 48.8 mm
- net /P1: track 0.00 -> 48.8 mm
- net /P5: track 0.00 -> 30.5 mm
- net /P2: track 0.00 -> 30.2 mm
- net GND: track 0.00 -> 15.6 mm
- net /P4: track 0.00 -> 12.8 mm
- net /P3: track 0.00 -> 12.0 mm
Other:
- board text added: "PCB1008_Knob8Vert_2017-08-01 github.com/Believotron/BelievotronWanderlustHardware"
- board text removed: "PCB1008_Knob8Vert_2017-07-28 github.com/Believotron/BelievotronWanderlustHardware"
