File: Beta1/PCB1008_Knob8_Vert/PCB1008-Knob8_Vert.kicad_pcb (KiCad board)
At the start: 2 copper layers, 160 x 15.9 mm, 18 parts, among them J0 CON_1x4, J1 CON_1x4, U1000 MCP3008T-I/SL

Commit message: Ready for fab
Other:
- board text added: "+3.3V"
- board text added: "CS"
- board text added: "GND"
- board text added: "PCB1008_Knob8Vert_2017-08-02 github.com/Believotron/BelievotronWanderlustHardware"
- board text added: "SPI_CLK"
- board text added: "SPI_MISO"
- board text added: "SPI_MOSI"
- board text removed: "PCB1008_Knob8Vert_2017-08-01 github.com/Believotron/BelievotronWanderlustHardware"
Changed lines of the file:
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@@
     (area -1.016 -63.02 185.860001 1.075)
     (thickness 1.6)
-    (drawings 18)
+    (drawings 26)
     (tracks 147)
     (zones 0)
@@
       (drillshape 0)
       (scaleselection 1)
-      (outputdirectory Output/PCB1005_2017-07-17_Gerbers/))
+      (outputdirectory Output/PCB1008_Gerbers_2017-08-02/))
   )
   (net 0 "")
@@
     (fp_line (start 4.25 -3.45) (end 4.25 1.95) (layer F.SilkS) (width 0.15))
     (fp_line (start -4.25 -3.45) (end 4.25 -3.45) (layer F.SilkS) (width 0.15))
-    (fp_text user RK09Y11L0001 (at 0.25 2.9) (layer F.SilkS)
+    (fp_text user RK09Y11L0001 (at -0.508 2.9) (layer F.SilkS)
       (effects (font (size 1 1) (thickness 0.15)))
     )
@@
     )
   )
+  (gr_text +3.3V (at 16.256 -6.858 90) (layer F.SilkS)
+    (effects (font (size 0.6 0.6) (thickness 0.125)))
+  )
+  (gr_text CS (at 18.796 -6.858 90) (layer F.SilkS)
+    (effects (font (size 0.6 0.6) (thickness 0.125)))
+  )
+  (gr_text GND (at 21.336 -6.858 90) (layer F.SilkS)
+    (effects (font (size 0.6 0.6) (thickness 0.125)))
+  )
+  (gr_text GND (at 23.876 -6.858 90) (layer F.SilkS)
+    (effects (font (size 0.6 0.6) (thickness 0.125)))
+  )
+  (gr_text SPI_CLK (at 134.366 -7.874 90) (layer F.SilkS)
+    (effects (font (size 0.6 0.6) (thickness 0.125)))
+  )
+  (gr_text SPI_MOSI (at 136.906 -7.874 90) (layer F.SilkS)
+    (effects (font (size 0.6 0.6) (thickness 0.125)))
+  )
+  (gr_text SPI_MISO (at 139.446 -7.874 90) (layer F.SilkS)
+    (effects (font (size 0.6 0.6) (thickness 0.125)))
+  )
+  (gr_text GND (at 141.986 -6.604 90) (layer F.SilkS)
+    (effects (font (size 0.6 0.6) (thickness 0.125)))
+  )
   (gr_text "All R=10KΩ\nAll C=0.1uF" (at 50.8 -2.54) (layer F.SilkS)
     (effects (font (size 1 1) (thickness 0.15)) (justify left))
@@
     (effects (font (size 1.15 1.15) (thickness 0.15)))
   )
-  (gr_text "PCB1008_Knob8Vert_2017-08-01 \ngithub.com/Believotron/BelievotronWanderlustHardware\n" (at 96.52 -2.54) (layer F.SilkS)
+  (gr_text "PCB1008_Knob8Vert_2017-08-02\ngithub.com/Believotron/BelievotronWanderlustHardware\n" (at 96.52 -2.54) (layer F.SilkS)
     (effects (font (size 0.8 0.8) (thickness 0.15)) (justify left))
   )
