File: Beta1/PCB1009_OLED_RISER/PCB1009_OLED_RISER.sch (KiCad schematic (older format))
At the start: 34 parts, among them J1 Axoloti_40Pin, U10 OLED_128x32_I2C, U1000 MCP3008T-I/SL, U2 MCP3008T-I/SL, U20 OLED_128x32_I2C, U30 OLED_128x32_I2C, U40 OLED_128x32_I2C, U5 I2C_1x4MUX_TCA9546A

Commit message: Creating 3D models
Parts:
- removed C1000, C2: 0.1u, Capacitors_SMD:C_0603, symbol C
- removed J1: Axoloti_40Pin, Liberry:Axoloti-40x1_slim, symbol Axoloti_40Pin
- removed JOY0, JOY1, JOY2, JOY3: XYJOY_Alps, Liberry:JOY_ALPS_RKJXV1224005, symbol XYJOY_Alps
- removed RV0, RV1, RV2, RV3, RV4, RV5, RV6, RV7: POT, Liberry:RV09AF-40-20K-B10K, symbol POT
- removed U1000, U2: MCP3008T-I/SL, Liberry:SOIC-16, symbol MCP3008T-I/SL
- added J0, J1: CON_1x4, Liberry:HEADER_0.1x4_SMT_VERT_SAMTECTSM-104-03-T-SV, symbol CON_1x4
Connections:
- net labels removed: CS_0_7, CS_8_15, JOY_0_0, JOY_0_1, JOY_0_SW, JOY_1_0, JOY_1_1, JOY_1_SW, JOY_2_0, JOY_2_1, JOY_2_SW, JOY_3_0, JOY_3_1, JOY_3_SW, P0, P1, P2, P3, P4, P5, P6, P7, SPI_CLK, SPI_MISO, SPI_MOSI, VOLUME
- wire segments 200 -> 74

Commit message: Finished routing
Changed lines of the file:
@@
 LIBS:Zilog
 LIBS:believotron_wanderlust
+LIBS:PCB1009_OLED_RISER-cache
 EELAYER 25 0
 EELAYER END
@@
 $EndComp
 Wire Wire Line
-	17900 5350 18100 5350
-Wire Wire Line
-	18100 5350 18100 5950
-Wire Wire Line
 	17900 5500 18100 5500
 Connection ~ 18100 5500
@@
 	17900 5800 18100 5800
 Connection ~ 18100 5800
+Wire Wire Line
+	18100 5500 18100 5950
+Wire Wire Line
+	17900 5350 19100 5350
+Text Label 17950 5350 0    60   ~ 0
+!OLED_RESET
 $EndSCHEMATC
