File: Beta1/PCB1009_OLED_RISER/PCB1009_OLED_RISER.kicad_pcb (KiCad board)
At the start: 2 copper layers, 160 x 60.2 mm, 45 parts, among them J1 Axoloti_40Pin, U10 OLED_128x32_I2C, U1000 MCP3008T-I/SL, U2 MCP3008T-I/SL, U20 OLED_128x32_I2C, U30 OLED_128x32_I2C, U40 OLED_128x32_I2C, U5 I2C_1x4MUX_TCA9546A

Commit message: Rough placement WIP
Parts:
- removed C1000, C2: 0.1u, Capacitors_SMD:C_0603
- removed JOY0, JOY1, JOY2, JOY3: XYJOY_Alps, Liberry:JOY_ALPS_RKJXV1224005
- removed the REF** at (156.5, -3.00)
- removed the REF** at (54.0, -52.2)
- removed the REF** at (44.0, -22.2)
- removed the REF** at (3.50, -3.00)
- removed the REF** at (3.50, -22.2)
- removed the REF** at (156.5, -22.2)
- removed the REF** at (156.5, -52.2)
- removed RV0, RV1, RV2, RV3, RV4, RV5, RV6, RV7: POT, Liberry:RV09AF-40-20K-B10K
- removed U1000, U2: MCP3008T-I/SL, Liberry:SOIC-16
- added J0: CON_1x4, Liberry:HEADER_0.1x4_SMT_VERT_SAMTECTSM-104-03-T-SV, B.Cu at (12.7, -5.08)
- C1, RC0, RC10, RC20, RC30, RC40, RD0, RD10, RD20, RD30, RD40, REF**, RR0, U5: moved to B.Cu
- J1: value Axoloti_40Pin -> CON_1x4; footprint Liberry:Axoloti-40x1_slim -> Liberry:HEADER_0.1x4_SMT_VERT_SAMTECTSM-104-03-T-SV; moved to B.Cu
- REF** (x2): moved to F.Cu
- moved REF** 176.7 mm to (-15.7, -23.1)
- moved REF** 169.2 mm to (-10.4, -38.1)
- moved J1 95.3 mm to (147.3, -5.08), turned to 90 degrees
- moved REF** 52.8 mm to (-8.13, -11.4)
- moved REF** 49.8 mm to (-9.91, -30.5)
- moved RC10 49.0 mm to (6.35, -6.35)
- moved RC20 49.0 mm to (45.7, -6.35)
- moved RC30 49.0 mm to (85.1, -6.35)
- moved RC40 49.0 mm to (124.5, -6.35)
- moved RD10 49.0 mm to (6.35, -8.89)
- moved RD20 49.0 mm to (45.7, -8.89)
- moved RD30 49.0 mm to (85.1, -8.89)
- moved RD40 49.0 mm to (124.5, -8.89)
- moved U10 49.0 mm to (2.54, -8.89)
- moved U20 49.0 mm to (41.9, -8.89)
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Connections:
- J1 pad 1: +3V3 -> GND
- J1 pad 2: /CS_8_15 -> GND
- J1 pad 3: /CS_0_7 -> GND
- J1 pad 4: /I2C_SCL -> GND
Routing:
- net +3V3: track 623.0 -> 0.00 mm, vias 7 -> 0
- net GND: track 475.0 -> 0.00 mm, vias 10 -> 0
- net /JOY_0_0: track 140.1 -> 0.00 mm, vias 1 -> 0
- net /JOY_0_1: track 124.7 -> 0.00 mm, vias 1 -> 0
- net /I2C_SDA3: track 104.9 -> 0.00 mm, vias 2 -> 0
- net /I2C_SCL3: track 103.0 -> 0.00 mm, vias 2 -> 0
- net /JOY_1_0: track 92.9 -> 0.00 mm, vias 1 -> 0
- net /SPI_CLK: track 87.1 -> 0.00 mm
- net /CS_8_15: track 84.1 -> 0.00 mm, vias 3 -> 0
- net /SPI_MISO: track 83.7 -> 0.00 mm, vias 4 -> 0
- net /P0: track 80.3 -> 0.00 mm, vias 1 -> 0
- net /SPI_MOSI: track 79.8 -> 0.00 mm, vias 4 -> 0
- net /JOY_1_1: track 76.9 -> 0.00 mm, vias 1 -> 0
- net /JOY_0_SW: track 76.3 -> 0.00 mm, vias 1 -> 0
- net /!OLED_RESET: track 71.2 -> 0.00 mm, vias 3 -> 0
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Other:
- board size 160 x 60.2 mm -> 160 x 10.2 mm
- board text removed: "MCP3008T-I/SL"
- board text removed: "RKJXV1224005"
- board text removed: "RV09AF-40-20K-B10K"

Commit message: Finished routing
Connections:
- J1 pad 1: GND -> /!OLED_RESET
Routing:
- net +3V3: track 0.00 -> 183.5 mm, vias 0 -> 8
- net /!OLED_RESET: track 0.00 -> 138.9 mm
- net /I2C_SCL3: track 0.00 -> 94.9 mm, vias 0 -> 2
- net /I2C_SDA3: track 0.00 -> 93.3 mm, vias 0 -> 1
- net /I2C_SCL2: track 0.00 -> 54.6 mm
- net /I2C_SDA2: track 0.00 -> 53.8 mm, vias 0 -> 2
- net /I2C_SCL0: track 0.00 -> 35.8 mm, vias 0 -> 1
- net /I2C_SDA0: track 0.00 -> 30.1 mm
- net /I2C_SCL: track 0.00 -> 24.9 mm
- net /I2C_SDA: track 0.00 -> 17.2 mm
- net /I2C_SDA1: track 0.00 -> 12.8 mm
- net /I2C_SCL1: track 0.00 -> 11.3 mm
- net GND: track 0.00 -> 6.69 mm, vias 0 -> 2

Commit message: Ready for fab
Parts:
- removed the REF** at (-8.13, -11.4)
- moved REF** 84.6 mm to (66.0, -1.91)
- moved REF** 79.1 mm to (66.0, -8.26)
- moved REF** 30.6 mm to (6.35, -1.91)
Routing:
- net GND: track 6.69 -> 132.8 mm, vias 2 -> 5
- net /!OLED_RESET: track 138.9 -> 142.0 mm
- net /I2C_SCL2: track 54.6 -> 53.1 mm
- net /I2C_SDA3: track 93.3 -> 94.4 mm
- net +3V3: track 183.5 -> 183.0 mm, vias 8 -> 9
Other:
- board text added: "PCB1009_OLED_RISER_2017-08-02 github.com/Believotron/BelievotronWanderlustHardware"
- board text removed: "PCB1005_KnobCore_2017-07-17 github.com/Believotron/BelievotronWanderlustHardware"
