File: Beta1/PCB1008_Knob8_Riser/PCB1008_Knob8_Riser.sch (KiCad schematic (older format))
At the start: 41 parts, among them J0-0 CONN_01X01, J0-1 CONN_01X01, J0-2 CONN_01X01, J0-3 CONN_01X01, J0-4 CONN_01X01, J0-5 CONN_01X01, J1 Axoloti_40Pin, J2 FPC_20POS, U1 MCP3008T-I/SL, U10 OLED_128x32_I2C, U2 MCP3008T-I/SL, U20 OLED_128x32_I2C, U3 I2C_1x4MUX_TCA9546A, U30 OLED_128x32_I2C, U40 OLED_128x32_I2C

Commit message: Removed Joysticks / OLED. Read for fab
Parts:
- removed C2, C3: 0.1u, Capacitors_SMD:C_0603, symbol C
- removed J1: Axoloti_40Pin, Liberry:Axoloti-40x1_slim, symbol Axoloti_40Pin
- removed J2: FPC_20POS, Liberry:FFC_1MM_20POS_MOLEX_52271-2079, symbol FPC_20POS
- removed JOY0, JOY1, JOY2, JOY3: XYJOY_Alps, Liberry:JOY_ALPS_RKJXV1224005, symbol XYJOY_Alps
- removed RC0, RC10, RC20, RC30, RC40, RD0, RD10, RD20, RD30, RD40, RR0: 10K, Resistors_SMD:R_0603, symbol R
- removed U10, U20, U30, U40: OLED_128x32_I2C, Liberry:OLED_128x32, symbol OLED_128x32_I2C
- removed U2: MCP3008T-I/SL, Liberry:SOIC-16, symbol MCP3008T-I/SL
- removed U3: I2C_1x4MUX_TCA9546A, Liberry:SOIC-16_1.27x5.4, symbol I2C_1x4MUX_TCA9546A
Connections:
- net labels removed: !OLED_RESET, ANALOG_OUT, CS_8_15, I2C_SCL, I2C_SCL0, I2C_SCL1, I2C_SCL2, I2C_SCL3, I2C_SDA, I2C_SDA0, I2C_SDA1, I2C_SDA2, I2C_SDA3, JOY_0_0, JOY_0_1, JOY_0_SW, JOY_1_0, JOY_1_1, JOY_1_SW, JOY_2_0, JOY_2_1, JOY_2_SW, JOY_3_0, JOY_3_1, JOY_3_SW, RX, TX, VOLUME
- wire segments 234 -> 53
Other:
- note removed: "PC0"
- note removed: "PC1"
- note removed: "PC2"
- note removed: "PC3"
- note removed: "PC4"
